Commit message: chore: publish complete Stage-1A portable runtime closure

File: source/data_collection/config/robot_cfg/G2/G2_omnipicker_fixed_dual.urdf (robot description, URDF)
Before this commit: robot genie, 58 links, 57 joints
Joints:
- joint arm_l_end_joint: origin xyz=0.095 0.0 0.0 rpy=3.1416 -1.5708 0 -> xyz=0.088 0.0 0.0 rpy=3.1416 -1.5708 0
- joint arm_r_end_joint: origin xyz=0.095 0.0 0.0 rpy=3.141592653589793 -1.5707963267948966 0 -> xyz=0.088 0.0 0.0 rpy=3.141592653589793 -1.5707963267948966 0
- joint idx52_gripper_l_center_joint: origin xyz=0.0 0.0 0.13008 rpy=0 0 -1.5707963267948966 -> xyz=0.0 0.0 0.14308 rpy=0 0 -1.5707963267948966
- joint idx92_gripper_r_center_joint: origin xyz=0.0 0.0 0.13008 rpy=0 0 -1.5707963267948966 -> xyz=0.0 0.0 0.14308 rpy=0 0 -1.5707963267948966
